File: DC_MOTOR.kicad_sch (KiCad schematic)
At the start: 6 parts, among them J5 Conn_01x04, U4 L293D

Commit message: Backups and updates
Parts:
- C6: value C_Small -> 100NF
- R11, R12: value R_Small -> 10K
Changed lines of the file:
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@@
       (effects (font (size 1.27 1.27)) (justify left))
     )
-    (property "Value" "R_Small" (id 1) (at 85.09 100.3299 0)
+    (property "Value" "10K" (id 1) (at 85.09 100.3299 0)
       (effects (font (size 1.27 1.27)) (justify left))
     )
@@
       (effects (font (size 1.27 1.27)) (justify left))
     )
-    (property "Value" "R_Small" (id 1) (at 85.09 90.1699 0)
+    (property "Value" "10K" (id 1) (at 85.09 90.1699 0)
       (effects (font (size 1.27 1.27)) (justify left))
     )
@@
       (effects (font (size 1.27 1.27)) (justify left))
     )
-    (property "Value" "C_Small" (id 1) (at 127 68.5862 0)
+    (property "Value" "100NF" (id 1) (at 127 68.5862 0)
       (effects (font (size 1.27 1.27)) (justify left))
     )
