File: POWER.kicad_sch (KiCad schematic)
At the start: 11 parts, among them J4 VIN_CONN, U2 AMS1117-3.3, U3 LM2596T-ADJ

Commit message: Backups and updates
Parts:
- C1: value C_Polarized -> 470uF
- C4: value C_Polarized -> 220uF
- R3: value R_Small -> 3K
- R4: value R_Small -> 1K
Changed lines of the file:
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@@
   (symbol (lib_id "Device:C_Polarized") (at 107.315 72.39 0) (unit 1)
     (in_bom yes) (on_board yes) (fields_autoplaced)
-    (property "Reference" "C1" (id 0) (at 111.125 70.2309 0)
-      (effects (font (size 1.27 1.27)) (justify left))
-    )
-    (property "Value" "C_Polarized" (id 1) (at 111.125 72.7709 0)
+    (property "Reference" "C1" (id 0) (at 110.49 70.2309 0)
+      (effects (font (size 1.27 1.27)) (justify left))
+    )
+    (property "Value" "470uF" (id 1) (at 110.49 72.7709 0)
       (effects (font (size 1.27 1.27)) (justify left))
     )
@@
   (symbol (lib_id "Device:C_Polarized") (at 186.055 84.455 0) (unit 1)
     (in_bom yes) (on_board yes) (fields_autoplaced)
-    (property "Reference" "C4" (id 0) (at 189.865 82.2959 0)
-      (effects (font (size 1.27 1.27)) (justify left))
-    )
-    (property "Value" "C_Polarized" (id 1) (at 189.865 84.8359 0)
+    (property "Reference" "C4" (id 0) (at 189.23 82.2959 0)
+      (effects (font (size 1.27 1.27)) (justify left))
+    )
+    (property "Value" "220uF" (id 1) (at 189.23 84.8359 0)
       (effects (font (size 1.27 1.27)) (justify left))
     )
@@
       (effects (font (size 1.27 1.27)) (justify left))
     )
-    (property "Value" "R_Small" (id 1) (at 211.455 89.5349 0)
+    (property "Value" "1K" (id 1) (at 211.455 89.5349 0)
       (effects (font (size 1.27 1.27)) (justify left))
     )
@@
       (effects (font (size 1.27 1.27)) (justify left))
     )
-    (property "Value" "R_Small" (id 1) (at 211.455 81.9149 0)
-      (effects (font (size 1.27 1.27)) (justify left))
-    )
+    (property "Value" "3K" (id 1) (at 211.455 81.9149 0)
+      (effects (font (size 1.27 1.27)) (justify left))
+    )
