File: mark_1.kicad_pcb (KiCad board)
At the start: 2 copper layers, 100.3 x 65.7 mm, 44 parts, among them J1 Conn_01x03, J10 MCU_PROG, J11 Conn_01x04, J12 MCU_PROG, J2 Conn_01x02, J3 Conn_01x05, J4 VIN_CONN, J5 Conn_01x04, J7 Conn_01x04, J8 MCU_PROG, J9 Conn_01x04, SW1 SW_Push, U1 ESP32-S2-WROOM, U2 AMS1117-3.3, U3 LM2596T-ADJ, U4 L293D

Commit message: Backups and updates
Parts:
- C1: value C_Polarized -> 470uF
- C4: value C_Polarized -> 220uF
- C6: value C_Small -> 100NF
- R11, R12: value R_Small -> 10K
- R3: value R_Small -> 3K
- R4: value R_Small -> 1K
Changed lines of the file:
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@@
       (effects (font (size 1 1) (thickness 0.15)))
     )
-    (fp_text value "C_Small" (at 0 1.68 90) (layer "F.Fab")
+    (fp_text value "100NF" (at 0 1.68 90) (layer "F.Fab")
       (effects (font (size 1 1) (thickness 0.15)))
     )
@@
     (pad "2" smd rect (at -3.975 2.25 90) (size 1.55 1.3) (layers "F.Cu" "F.Paste" "F.Mask")
       (net 45 "Net-(R1-Pad2)") (pinfunction "2") (pintype "passive"))
-    (model "${KICAD6_3DMODEL_DIR}/Button_Switch_SMD.3dshapes/SW_PUSH_6mm_H9.5mm.wrl"
+    (model "${KICAD6_3DMODEL_DIR}/Button_Switch_SMD.3dshapes/SW_SPST_PTS645.step"
       (offset (xyz 0 0 0))
       (scale (xyz 1 1 1))
@@
     (pad "16" thru_hole oval (at 12.7 0 90) (size 1.6 1.6) (drill 0.8) (layers *.Cu *.Mask)
       (net 35 "Y_DIR") (pinfunction "DIR") (pintype "input"))
-    (model "${KICAD6_3DMODEL_DIR}/Module.3dshapes/Pololu_Breakout-16_15.2x20.3mm.wrl"
-      (offset (xyz 0 0 0))
-      (scale (xyz 1 1 1))
-      (rotate (xyz 0 0 0))
+    (model "${M3_3D}/DRV8825_STEPPER_MOTOR_DRIVER_CARRIER.step"
+      (offset (xyz 6.5 -9 3.5))
+      (scale (xyz 1 1 1))
+      (rotate (xyz -90 0 -180))
     )
   )
@@
     (pad "16" thru_hole oval (at 12.7 0 90) (size 1.6 1.6) (drill 0.8) (layers *.Cu *.Mask)
       (net 25 "X_DIR") (pinfunction "DIR") (pintype "input"))
-    (model "${KICAD6_3DMODEL_DIR}/Module.3dshapes/Pololu_Breakout-16_15.2x20.3mm.wrl"
-      (offset (xyz 0 0 0))
-      (scale (xyz 1 1 1))
-      (rotate (xyz 0 0 0))
+    (model "${M3_3D}/DRV8825_STEPPER_MOTOR_DRIVER_CARRIER.step"
+      (offset (xyz 6.5 -9 3.5))
+      (scale (xyz 1 1 1))
+      (rotate (xyz -90 0 -180))
     )
   )
@@
       (effects (font (size 1 1) (thickness 0.15)))
     )
-    (fp_text value "R_Small" (at 0 1.43 90) (layer "F.Fab")
+    (fp_text value "10K" (at 0 1.43 90) (layer "F.Fab")
       (effects (font (size 1 1) (thickness 0.15)))
     )
@@
     (pad "16" thru_hole oval (at 12.7 0 90) (size 1.6 1.6) (drill 0.8) (layers *.Cu *.Mask)
       (net 14 "Z_DIR") (pinfunction "DIR") (pintype "input"))
-    (model "${KICAD6_3DMODEL_DIR}/Module.3dshapes/Pololu_Breakout-16_15.2x20.3mm.wrl"
-      (offset (xyz 0 0 0))
-      (scale (xyz 1 1 1))
-      (rotate (xyz 0 0 0))
+    (model "${M3_3D}/DRV8825_STEPPER_MOTOR_DRIVER_CARRIER.step"
+      (offset (xyz 6.5 -9 3.5))
+      (scale (xyz 1 1 1))
+      (rotate (xyz -90 0 -180))
     )
   )
@@
       (effects (font (size 1 1) (thickness 0.15)) (justify mirror))
     )
-    (fp_text value "R_Small" (at 0 -1.65) (layer "B.Fab")
+    (fp_text value "1K" (at 0 -1.65) (layer "B.Fab")
       (effects (font (size 1 1) (thickness 0.15)) (justify mirror))
     )
@@
       (effects (font (size 1 1) (thickness 0.15)) (justify mirror))
     )
-    (fp_text value "C_Polarized" (at 0 -5.2) (layer "B.Fab")
+    (fp_text value "220uF" (at 0 -5.2) (layer "B.Fab")
       (effects (font (size 1 1) (thickness 0.15)) (justify mirror))
     )
@@
       (effects (font (size 1 1) (thickness 0.15)) (justify mirror))
     )
-    (fp_text value "C_Polarized" (at 0 -5.2) (layer "B.Fab")
+    (fp_text value "470uF" (at 0 -5.2) (layer "B.Fab")
       (effects (font (size 1 1) (thickness 0.15)) (justify mirror))
     )
@@
       (effects (font (size 1 1) (thickness 0.15)) (justify mirror))
     )
-    (fp_text value "R_Small" (at 0 -1.65 90) (layer "B.Fab")
+    (fp_text value "3K" (at 0 -1.65 90) (layer "B.Fab")
       (effects (font (size 1 1) (thickness 0.15)) (justify mirror))
     )
@@
       (effects (font (size 1 1) (thickness 0.15)) (justify mirror))
     )
-    (fp_text value "R_Small" (at 0 -1.43) (layer "B.Fab")
+    (fp_text value "10K" (at 0 -1.43) (layer "B.Fab")
       (effects (font (size 1 1) (thickness 0.15)) (justify mirror))
     )
@@
     (pad "2" smd roundrect (at 4.95 0 90) (size 2.9 5.4) (layers "B.Cu" "B.Paste" "B.Mask") (roundrect_rratio 0.25)
       (net 2 "+5V") (pinfunction "2") (pintype "input"))
-    (model "${KICAD6_3DMODEL_DIR}/Inductor_SMD.3dshapes/L_12x12mm_H6mm.wrl"
-      (offset (xyz 0 0 0))
-      (scale (xyz 1 1 1))
-      (rotate (xyz 0 0 0))
-    )
-  )
+    (model "${M3_3D}/CDRH74 7.3x7.3x4.5 mm.stp"
+      (offset (xyz 0 0 0))
+      (scale (xyz 2 2 2))
+      (rotate (xyz -90 0 0))
+    )
+  )
